Commit message: Day 23

File: src/my_robot_description/urdf/robot_base.xacro (robot description, xacro)
@@ -23,4 +23,5 @@
       </material>
     </visual>
+    <!-- ===== Collision 1: 메인 프레임 ===== -->
     <collision>
       <origin xyz="0.0 0.0 ${frame_height/2}" rpy="0.0 0.0 0.0"/>
@@ -29,4 +30,42 @@
       </geometry>
     </collision>
+    <!-- ===== Collision 2: LiDAR 폴 ===== -->
+    <collision>
+      <origin xyz="${lidar_x} 0.0 ${frame_height + 0.075}" rpy="0.0 0.0 0.0"/>
+      <geometry>
+        <box size="0.030 0.030 0.150"/>
+      </geometry>
+    </collision>
+    <!--
+      LiDAR 폴: 20×20mm 프로파일이지만 약간 여유있게 30×30
+      높이: 150mm
+      Z 중심: 243(상판) + 75(폴 절반) = 318mm
+      왜 추가?
+        폴이 프레임 위로 150mm 돌출
+        → Nav2 costmap에서 이 영역을 고려해야 → 좁은 통로에서 폴이 걸릴 수 있음
+    -->
+    <!-- ===== Collision 3: LiDAR 본체 + 마운트 ===== -->
+    <collision>
+      <origin xyz="${lidar_x} 0.0 ${lidar_z}" rpy="0.0 0.0 0.0"/>
+      <geometry>
+        <cylinder radius="0.045" length="0.060"/>
+      </geometry>
+    </collision>
+    <!--
+      LiDAR 마운트판(80×80) + 센서(Ø70×41) 통합
+      반지름 45mm, 높이 60mm으로 근사
+        → 실제 lidar_link에도 collision이 있지만 base_link 쪽에도 마운트 영역을 커버
+    -->
+     <!-- ===== Collision 4: 카메라 마운트 (전방 돌출) ===== -->
+    <collision>
+      <origin xyz="${frame_length/2 + 0.015} 0.0 ${camera_z}" rpy="0.0 0.0 0.0"/>
+      <geometry>
+        <box size="0.060 0.100 0.035"/>
+      </geometry>
+    </collision>
+    <!--
+      카메라+마운트가 프레임 전방으로 돌출!
+      프레임 끝(175mm) + 마운트(~30mm) 영역 → 벽에 접근할 때 카메라가 먼저 부딪히도록!
+    -->
     <inertial>
       <origin xyz="${base_com_x} ${base_com_y} ${base_com_z}"

File: src/my_robot_description/urdf/robot_gazebo.xacro (robot description, xacro)
@@ -10,4 +10,6 @@
   <gazebo>
     <plugin name="diff_drive" filename="libgazebo_ros_diff_drive.so">
+      <!-- 바퀴 쌍 수: 1 (2륜 차동 구동) -->
+      <num_wheel_pairs>1</num_wheel_pairs>
       <left_joint>left_wheel_joint</left_joint>
       <right_joint>right_wheel_joint</right_joint>
@@ -28,5 +30,29 @@
       <publish_odom_tf>true</publish_odom_tf>
       <publish_wheel_tf>false</publish_wheel_tf>
+      <odometry_source>1</odometry_source>
+      <!--
+        오도메트리 계산 소스:
+          0: 엔코더 (Joint 위치에서 계산) ← 더 현실적!
+          1: World (Gazebo 내부 위치에서 계산) ← Ground Truth!
+        차이:
+          소스 0 (엔코더):
+            → 바퀴 회전량으로 계산 → 슬립이 있으면 부정확!
+            → 실제 로봇과 동일한 오차 패턴!
+            → Sim-to-Real 테스트에 적합!
+          소스 1 (World):
+            → Gazebo가 알고 있는 정확한 위치 사용
+            → 오차 없음 = Ground Truth!
+            → 알고리즘 검증에 유용 (비교 기준)
+        ⭐ 개발 단계에서는 1 (정확한 odom으로 빠른 개발)
+          Sim-to-Real 단계에서는 0 (현실적 odom으로 테스트)
+      -->
       <update_rate>50.0</update_rate>
+    </plugin>
+  </gazebo>
+   <gazebo>
+    <plugin name="joint_state_publisher" filename="libgazebo_ros_joint_state_publisher.so">
+      <update_rate>50</update_rate>
+      <joint_name>left_wheel_joint</joint_name>
+      <joint_name>right_wheel_joint</joint_name>
     </plugin>
   </gazebo>
@@ -35,5 +61,5 @@
     <sensor name="lidar" type="ray">
       <always_on>true</always_on>
-      <visualize>true</visualize>
+      <visualize>false</visualize>
       <update_rate>5.5</update_rate>
       <ray>
@@ -67,4 +93,11 @@
   </gazebo>
   <!-- Depth Camera Sensor -->
+  <!--RealSense D435 깊이 노이즈 특성: Stereo 기반 → 깊이 오차가 거리의 제곱에 비례
+    σ_depth ≈ z² × baseline⁻¹ × focal_length⁻¹ × σ_disparity
+    근거리(1m): σ ≈ 2~5mm
+    중거리(3m): σ ≈ 20~40mm
+    원거리(5m): σ ≈ 80~150mm
+    Gazebo는 거리 비례 노이즈를 직접 지원하지 않으므로 평균적인 값을 사용하거나 ROS 2 노드에서 후처리로 추가!
+  -->
   <gazebo reference="camera_link">
     <sensor name="depth_camera" type="depth">
@@ -83,4 +116,19 @@
           <far>10.0</far>
         </clip>
+        <noise>
+          <type>gaussian</type>
+          <mean>0.0</mean>
+          <stddev>0.007</stddev>
+          <!--
+            RGB 이미지 노이즈: σ = 0.007
+              → 픽셀 값(0~1 정규화)에 대한 표준편차
+              → 255 스케일에서: 0.007 × 255 ≈ 1.8
+              → 약 2 gray level의 노이즈
+              → 잘 조명된 실내에서의 일반적인 카메라 노이즈
+          -->
+        </noise>
+        <depth_camera>
+          <output>depths</output>
+        </depth_camera>
       </camera>
       <plugin name="depth_camera_controller" filename="libgazebo_ros_camera.so">
@@ -95,8 +143,32 @@
           ⚠️ camera_link가 아닌 camera_optical_frame → 이미지 데이터는 optical frame 기준으로 발행
         -->
+        <hack_baseline>0.07</hack_baseline>
+        <!--
+          hack_baseline: Stereo 베이스라인
+          D435: 50mm (IR 카메라 간 거리)
+            → 깊이 이미지의 노이즈 특성에 영향
+            → 0.07 (약간 더 넓게)
+        -->
+        <min_depth>0.1</min_depth>
+        <max_depth>10.0</max_depth>
+        <update_rate>30</update_rate>
       </plugin>
     </sensor>
   </gazebo>
   <!-- IMU Sensor -->
+  <!--
+      IMU 노이즈는 2가지 유형:
+      1. Rate Noise (White Noise): 매 측정마다 랜덤
+      2. Bias (Random Walk): 천천히 누적되는 체계적 오차
+      실제 BNO055 데이터시트:
+        Gyroscope:
+        Noise Density: 0.014 °/s/√Hz = 0.000244 rad/s/√Hz
+        → σ_rate = noise_density × √(bandwidth)
+        → bandwidth ≈ 100 Hz
+        → σ_rate = 0.000244 × √100 = 0.00244 rad/s
+      Accelerometer:
+        Noise Density: 150 μg/√Hz = 0.00147 m/s²/√Hz
+        → σ_rate = 0.00147 × √100 = 0.0147 m/s²
+-->
   <gazebo reference="imu_link">
     <sensor name="imu" type="imu">
@@ -104,13 +176,30 @@
       <update_rate>100.0</update_rate>
       <imu>
+        <!-- 각속도 (Gyroscope) 노이즈 -->
         <angular_velocity>
-          <x><noise type="gaussian"><mean>0.0</mean><stddev>0.0002</stddev></noise></x>
-          <y><noise type="gaussian"><mean>0.0</mean><stddev>0.0002</stddev></noise></y>
-          <z><noise type="gaussian"><mean>0.0</mean><stddev>0.0002</stddev></noise></z>
+          <x><noise type="gaussian"><mean>0.0</mean><stddev>0.0002</stddev><bias_mean>0.0000075</bias_mean><bias_stddev>0.0000008</bias_stddev></noise></x>
+          <!--
+            Bias Random Walk: 느리게 변하는 체계적 편향
+              → 시간이 지나면 측정값이 서서히 한쪽으로 치우침
+              → 이것이 IMU "드리프트"의 원인!
+              → BNO055 Fusion 모드는 드리프트가 매우 작음
+            bias_mean: 초기 편향의 평균
+            bias_stddev: 편향이 변하는 속도
+          -->
+          <y><noise type="gaussian"><mean>0.0</mean><stddev>0.0002</stddev><bias_mean>0.0000075</bias_mean><bias_stddev>0.0000008</bias_stddev></noise></y>
+          <z><noise type="gaussian"><mean>0.0</mean><stddev>0.0002</stddev><bias_mean>0.0000075</bias_mean><bias_stddev>0.0000008</bias_stddev></noise></z>
         </angular_velocity>
+        <!-- 선가속도 (Accelerometer) 노이즈 -->
         <linear_acceleration>
-          <x><noise type="gaussian"><mean>0.0</mean><stddev>0.017</stddev></noise></x>
-          <y><noise type="gaussian"><mean>0.0</mean><stddev>0.017</stddev></noise></y>
-          <z><noise type="gaussian"><mean>0.0</mean><stddev>0.017</stddev></noise></z>
+          <x><noise type="gaussian"><mean>0.0</mean><stddev>0.017</stddev><bias_mean>0.1</bias_mean><bias_stddev>0.001</bias_stddev></noise></x>
+          <!--
+            가속도계 바이어스:
+              → 중력 방향 감지에 영향
+              → 0.1 m/s² ≈ 10 mg의 초기 바이어스
+              → 실제 센서 캘리브레이션으로 줄일 수 있지만 완벽히 제거는 불가!
+              → 이것이 EKF에서 가속도계를 "장기 기준"으로만 사용하는 이유!
+          -->
+          <y><noise type="gaussian"><mean>0.0</mean><stddev>0.017</stddev><bias_mean>0.1</bias_mean><bias_stddev>0.001</bias_stddev></noise></y>
+          <z><noise type="gaussian"><mean>0.0</mean><stddev>0.017</stddev><bias_mean>0.1</bias_mean><bias_stddev>0.001</bias_stddev></noise></z>
         </linear_acceleration>
       </imu>

File: src/my_robot_description/urdf/robot_properties.xacro (robot description, xacro)
@@ -15,5 +15,5 @@
   <xacro:property name="frame_width" value="0.300"/>
   <!-- Z방향 240mm = 0.240m (높이) -->
-  <xacro:property name="frame_height" value="0.240"/>
+  <xacro:property name="frame_height" value="0.243"/>
   <!-- 지상고 57.5mm = 0.0575m -->
   <xacro:property name="ground_clearance" value="0.0575"/>
@@ -29,7 +29,26 @@
   <!-- 바퀴 Z 오프셋: 하판 아래 25mm -->
   <xacro:property name="wheel_z_offset" value="-0.025"/>
+  <!-- 캐스터 치수 -->
+  <!--캐스터 볼 반지름: 12.5mm-->
+  <xacro:property name="caster_radius" value="0.0125"/>
+  <!--
+    계산:
+      바퀴 바닥 → 지면: Z = -0.0575 (base_link 기준)
+      바퀴 중심: Z = -0.045
+      바퀴 반지름: 32.5mm
+        → 지면 Z = -0.005(탭) -0.020(클램프 중심) - 0.0325 = -0.0575 (base_link 기준)
+      캐스터 볼 중심도 지면에서 볼 반지름만큼 위에 있어야 함
+        캐스터 Z = -0.0575 + 0.012.5 = -0.045
+  -->
+  <!-- 전방 100mm (프레임 앞쪽) -->
+  <xacro:property name="caster_x_offset" value="0.100"/>
+  <!-- 좌우 캐스터 사이 거리: 280mm (Y=±140mm) -->
+  <xacro:property name="caster_y_separation" value="0.280"/>
+  <!-- base_link 원점(하판 바닥)에서 캐스터 볼 중심까지: 45mm -->
+  <xacro:property name="caster_z_offset" value="-0.045"/>
   <!-- 질량 (kg) -->
-  <xacro:property name="base_mass" value="4.79"/>
+  <xacro:property name="base_mass" value="4.73"/>
   <xacro:property name="wheel_mass" value="0.080"/>
+  <xacro:property name="caster_mass" value="0.030"/>
   <xacro:property name="lidar_mass" value="0.170"/>
   <xacro:property name="camera_mass" value="0.072"/>
@@ -76,3 +95,12 @@
     </inertial>
   </xacro:macro>
+  <!-- 구체 관성 매크로 (기존에 없었으므로 추가) -->
+  <xacro:macro name="sphere_inertia" params="m r">
+    <inertial>
+      <mass value="${m}"/>
+      <inertia ixx="${(2/5)*m*r*r}" ixy="0.0" ixz="0.0"
+               iyy="${(2/5)*m*r*r}" iyz="0.0"
+               izz="${(2/5)*m*r*r}"/>
+    </inertial>
+  </xacro:macro>
 </robot>

File: src/my_robot_description/urdf/robot_wheels.xacro (robot description, xacro)
@@ -1,9 +1,7 @@
 <?xml version="1.0"?>
-<!--
-  ⭐ left_wheel과 right_wheel은 Y좌표 부호만 다름
-    → 매크로 1개로 양쪽 바퀴를 모두 생성
--->
 <robot xmlns:xacro="http://www.ros.org/wiki/xacro">
+  <!-- ============================================ -->
   <!-- 바퀴 매크로 정의 -->
+  <!-- ============================================ -->
   <xacro:macro name="wheel" params="prefix y_reflect">
     <!--
@@ -11,11 +9,11 @@
         prefix: "left" 또는 "right" (이름 접두사)
         y_reflect: +1 (왼쪽) 또는 -1 (오른쪽) (Y방향 반전)
-      이 매크로를 호출하면 Joint + Link가 자동 생성
+        이 매크로를 호출하면 Joint + Link가 자동 생성
     -->
     <joint name="${prefix}_wheel_joint" type="continuous">
       <!--
         ${prefix}_wheel_joint
-            → "left_wheel_joint" 또는 "right_wheel_joint"
-            → 문자열 조합이 가능
+          → "left_wheel_joint" 또는 "right_wheel_joint"
+          → 문자열 조합이 가능
       -->
       <parent link="base_link"/>
@@ -26,16 +24,31 @@
           left:  +1 * 0.345/2 = +0.172.5
           right: -1 * 0.345/2 = -0.172.5
-            → 하나의 수식으로 양쪽 모두 처리!
       -->
       <axis xyz="0 1 0"/>
+      <!-- ⭐ 감쇠 추가! -->
+      <dynamics damping="0.1" friction="0.05"/>
+      <!--
+        damping = 0.1: 속도 1 rad/s에서 0.1 N·m의 저항 토크 (바퀴가 돌 때 저항을 줌. 속도가 빠를수록 저항 토크가 커짐.)
+          바퀴가 330 RPM(=34.6 rad/s)일 때: 저항 토크 = 0.1 × 34.6 = 3.46 N·m
+          → 모터 토크(1.5 N·m)보다 큼?
+          → diff_drive 플러그인은 max_wheel_torque를 적용하므로
+            모터가 이 저항을 이길 수 있도록 max_wheel_torque ≥ 필요 토크 + 감쇠 토크!
+          ⚠️ max_wheel_torque가 너무 작으면 damping 때문에 바퀴가 안 돌 수 있음
+        friction = 0.05: 정지 시 0.05 N·m의 고정 마찰 (바퀴가 멈춰 있을 때 "정지 마찰"을 줌.)
+          → 경사에서 굴러내려가지 않도록!
+          → 미세한 값이므로 동작에 큰 영향 없음
+      -->
+      <limit effort="5.0" velocity="40.0"/>
+      <!--
+        effort: 최대 토크 제한 (N·m)
+          5.0 N·m = JGB37-520 스톨 토크의 ~1/3 → 모터가 발휘할 수 있는 연속 토크
+        velocity: 최대 각속도 제한 (rad/s)
+          40.0 rad/s ≈ 382 RPM → 330 RPM(34.6 rad/s) + 여유
+        limit 태그의 역할: Gazebo가 이 한계를 넘지 않도록 제한 → 실제 모터의 물리적 한계를 시뮬에 반영
+      -->
     </joint>
     <link name="${prefix}_wheel">
       <visual>
         <origin xyz="0.0 0.0 0.0" rpy="${pi/2} 0.0 0.0"/>
-        <!--
-          ${pi/2} = 1.5708...
-            Xacro는 pi를 내장 상수로 제공
-            → 1.5708 하드코딩 불필요
-        -->
         <geometry>
           <cylinder radius="${wheel_radius}" length="${wheel_width}"/>
@@ -51,12 +64,8 @@
         </geometry>
       </collision>
-      <xacro:cylinder_inertia m="${wheel_mass}"
-                               r="${wheel_radius}"
-                               h="${wheel_width}"/>
-      <!--
-        ⭐ 관성 모멘트 매크로 호출 → robot_properties.xacro에서 정의한 매크로
-      -->
+      <xacro:cylinder_inertia m="${wheel_mass}" r="${wheel_radius}" h="${wheel_width}"/>
+      <!-- ⭐ 관성 모멘트 매크로 호출 → robot_properties.xacro에서 정의한 매크로 -->
     </link>
-    <!-- Gazebo 마찰 설정도 매크로 안에 -->
+    <!-- Gazebo 마찰 설정 -->
     <gazebo reference="${prefix}_wheel">
       <material>Gazebo/Black</material>
@@ -71,14 +80,91 @@
   <!--
     이 한 줄로 생성되는 것:
-    ✅ left_wheel_joint (continuous, Y=+0.155)
-    ✅ left_wheel (link with visual/collision/inertial)
-    ✅ Gazebo 마찰 설정
+      ✅ left_wheel_joint (continuous, Y=+0.172.5)
+      ✅ left_wheel (link with visual/collision/inertial)
+      ✅ Gazebo 마찰 설정
   -->
   <xacro:wheel prefix="right" y_reflect="-1"/>
   <!--
     이 한 줄로 생성되는 것:
-    ✅ right_wheel_joint (continuous, Y=-0.155)
-    ✅ right_wheel (link with visual/collision/inertial)
-    ✅ Gazebo 마찰 설정
+      ✅ right_wheel_joint (continuous, Y=-0.172.5)
+      ✅ right_wheel (link with visual/collision/inertial)
+      ✅ Gazebo 마찰 설정
   -->
+  <!-- ============================================ -->
+  <!-- 캐스터 매크로 정의 -->
+  <!-- ============================================ -->
+  <!--
+    설계 의도:
+      1. 물리적 지지력 제공 (로봇이 기울어지지 않음)
+      2. 극히 낮은 마찰 → diff_drive에 간섭 안 함
+      3. 구체라서 어느 방향으로든 자유롭게 굴러감
+    실제 볼 캐스터:
+      → 하우징 안에서 볼이 자유 회전
+      → 시뮬에서는 저마찰 구체로 동일한 효과
+  -->
+  <xacro:macro name="caster_wheel" params="prefix y_reflect">
+    <joint name="${prefix}_caster_joint" type="fixed">
+      <!--
+        type="fixed":
+          캐스터를 base_link에 고정!
+        왜 continuous가 아닌 fixed?
+          → 실제 볼 캐스터는 회전하지만 시뮬에서는 저마찰 구체가 지면 위에서 미끄러짐
+          → Joint을 추가하면 불필요한 복잡성만 늘어남
+          → fixed + 저마찰 = 업계 표준 패턴
+      -->
+      <parent link="base_link"/>
+      <child link="${prefix}_caster_link"/>
+      <origin xyz="${caster_x_offset} ${y_reflect * caster_y_separation / 2} ${caster_z_offset}" rpy="0.0 0.0 0.0"/>
+      <!--
+        left:  Y = +1 × 0.280/2 = +0.140
+        right: Y = -1 × 0.280/2 = -0.140
+        Z = -0.045 (지면 바로 위)
+      -->
+    </joint>
+    <link name="${prefix}_caster_link">
+      <visual>
+        <geometry>
+          <sphere radius="${caster_radius}"/>
+        </geometry>
+        <material name="dark_grey">
+          <color rgba="0.3 0.3 0.3 1.0"/>
+        </material>
+      </visual>
+      <collision>
+        <geometry>
+          <sphere radius="${caster_radius}"/>
+        </geometry>
+      </collision>
+      <xacro:sphere_inertia m="${caster_mass}" r="${caster_radius}"/>
+    </link>
+    <!-- Gazebo 마찰 설정 -->
+    <gazebo reference="${prefix}_caster_link">
+      <material>Gazebo/DarkGrey</material>
+      <mu1>0.001</mu1>
+      <mu2>0.001</mu2>
+      <!--
+        ⭐ 핵심: 마찰이 거의 0!
+        mu = 0.001:
+          구동 바퀴: mu = 1.0 (높은 마찰 = 접지력)
+          캐스터: mu = 0.001 (거의 무마찰 = 자유 미끄러짐)
+        왜?
+          차동 구동의 회전 원리:
+            좌우 바퀴 속도 차이 → 회전
+              이때 캐스터는 옆으로 미끄러져야 함!
+              캐스터 마찰이 높으면 → 회전 못 함!
+      -->
+      <kp>1000000.0</kp>
+      <kd>100.0</kd>
+      <!--
+        kp: 접촉 강성 (높아야 바닥을 안 뚫음)
+        kd: 접촉 감쇠 (바운스 방지)
+        kd를 10→100으로 올림:
+          캐스터가 작고 가벼워서 진동이 생기기 쉬움
+          감쇠를 높여서 안정화!
+      -->
+    </gazebo>    \
+  </xacro:macro>
+  <!-- 캐스터 매크로 호출 — 2개 생성! -->
+  <xacro:caster_wheel prefix="front_left" y_reflect="1"/>
+  <xacro:caster_wheel prefix="front_right" y_reflect="-1"/>
 </robot>
