Commit message: Day 50

File: src/my_robot_description/urdf/robot_gazebo.xacro (robot description, xacro)
@@ -100,6 +100,6 @@
     Gazebo는 거리 비례 노이즈를 직접 지원하지 않으므로 평균적인 값을 사용하거나 ROS 2 노드에서 후처리로 추가!
   -->
-  <gazebo reference="camera_link">
-    <sensor name="depth_camera" type="depth">
+  <gazebo reference="camera_color_frame">
+    <sensor type="camera" name="color_camera">
       <always_on>true</always_on>
       <visualize>false</visualize>
@@ -113,6 +113,6 @@
         </image>
         <clip>
-          <near>0.1</near>
-          <far>10.0</far>
+          <near>0.02</near>
+          <far>300</far>
         </clip>
         <noise>
@@ -128,29 +128,46 @@
           -->
         </noise>
-        <depth_camera>
-          <output>depths</output>
-        </depth_camera>
       </camera>
-      <plugin name="depth_camera_controller" filename="libgazebo_ros_camera.so">
+      <plugin name="camera_color" filename="libgazebo_ros_camera.so">
         <ros>
           <remapping>~/image_raw:=camera/color/image_raw</remapping>
-          <remapping>~/depth/image_raw:=camera/depth/image_rect_raw</remapping>
           <remapping>~/camera_info:=camera/color/camera_info</remapping>
-          <remapping>~/depth/camera_info:=camera/depth/camera_info</remapping>
-        </ros>
-        <frame_name>camera_optical_frame</frame_name>
-        <!--
-          ⚠️ camera_link가 아닌 camera_optical_frame → 이미지 데이터는 optical frame 기준으로 발행
-        -->
-        <hack_baseline>0.07</hack_baseline>
-        <!--
-          hack_baseline: Stereo 베이스라인
-          D435: 50mm (IR 카메라 간 거리)
-            → 깊이 이미지의 노이즈 특성에 영향
-            → 0.07 (약간 더 넓게)
-        -->
+        </ros>
+        <frame_name>camera_color_optical_frame</frame_name>
+      </plugin>
+    </sensor>
+  </gazebo>
+  <gazebo reference="camera_depth_frame">
+    <sensor type="depth" name="depth_camera">
+      <always_on>true</always_on>
+      <visualize>false</visualize>
+      <update_rate>30.0</update_rate>
+      <camera>
+        <horizontal_fov>1.5184</horizontal_fov>
+        <image>
+          <width>640</width>
+          <height>480</height>
+          <format>B8G8R8</format>
+          <!-- depth 센서도 내부적으로는 이미지 생성 -->
+        </image>
+        <clip>
+          <near>0.1</near>
+          <far>10.0</far>
+        </clip>
+        <noise>
+          <type>gaussian</type>
+          <mean>0.0</mean>
+          <stddev>0.005</stddev>
+        </noise>
+      </camera>
+      <plugin name="camera_depth" filename="libgazebo_ros_camera.so">
+        <ros>
+          <remapping>~/image_raw:=camera/depth/image_rect_raw</remapping>
+          <remapping>~/camera_info:=camera/depth/camera_info</remapping>
+          <remapping>~/points:=/camera/depth/color/points</remapping>
+        </ros>
+        <frame_name>camera_depth_optical_frame</frame_name>
         <min_depth>0.1</min_depth>
         <max_depth>10.0</max_depth>
-        <update_rate>30</update_rate>
       </plugin>
     </sensor>

File: src/my_robot_description/urdf/robot_sensors.xacro (robot description, xacro)
@@ -55,17 +55,35 @@
     → realsense2_camera 드라이버가 이걸 자동으로 발행하지만 시뮬에서는 직접 정의해야 할 수 있음
   -->
-  <joint name="camera_optical_joint" type="fixed">
+  <joint name="camera_color_joint" type="fixed">
     <parent link="camera_link"/>
-    <child link="camera_optical_frame"/>
+    <child link="camera_color_frame"/>
+    <origin xyz="0 0 0" rpy="0 0 0"/>
+  </joint>
+  <joint name="camera_color_optical_joint" type="fixed">
+    <parent link="camera_color_frame"/>
+    <child link="camera_color_optical_frame"/>
     <origin xyz="0.0 0.0 0.0" rpy="${-pi/2} 0.0 ${-pi/2}"/>
-    <!--
-      rpy 변환:
-        Roll = -π/2: Y→Z 변환
-        Yaw  = -π/2: X→Y 변환
-        결과: 로봇좌표 → 카메라 광학 좌표
-    -->
   </joint>
+  <joint name="camera_depth_joint" type="fixed">
+    <parent link="camera_link"/>
+    <child link="camera_depth_frame"/>
+    <origin xyz="0 0 0" rpy="0 0 0"/>
+  </joint>
+  <joint name="camera_depth_optical_joint" type="fixed">
+    <parent link="camera_depth_frame"/>
+    <child link="camera_depth_optical_frame"/>
+    <origin xyz="0.0 0.0 0.0" rpy="${-pi/2} 0.0 ${-pi/2}"/>
+  </joint>
+  <!--
+    rpy 변환:
+      Roll = -π/2: Y→Z 변환
+      Yaw  = -π/2: X→Y 변환
+      결과: 로봇좌표 → 카메라 광학 좌표
+  -->
   <!-- 가상 Link: 좌표 변환용, 물리적 실체 없음 -->
-  <link name="camera_optical_frame"/>
+  <link name="camera_color_frame"/>
+  <link name="camera_color_optical_frame"/>
+  <link name="camera_depth_frame"/>
+  <link name="camera_depth_optical_frame"/>
   <!-- IMU (BNO055) -->
   <joint name="imu_joint" type="fixed">

Commit message: Day 54

File: src/my_robot_description/urdf/robot_gazebo.xacro (robot description, xacro)
@@ -16,11 +16,6 @@
       <wheel_separation>${wheel_separation}</wheel_separation>
       <wheel_diameter>${wheel_radius * 2}</wheel_diameter>
-      <!--
-        ${wheel_radius * 2} = 0.0325 * 2 = 0.065
-        → 변수에 수식 적용!
-        → 직경 = 반지름 × 2
-      -->
-      <max_wheel_torque>5.0</max_wheel_torque>
-      <max_wheel_acceleration>2.0</max_wheel_acceleration>
+      <max_wheel_torque>10.0</max_wheel_torque>
+      <max_wheel_acceleration>1.0</max_wheel_acceleration>
       <command_topic>cmd_vel</command_topic>
       <odometry_topic>odom</odometry_topic>
@@ -30,5 +25,5 @@
       <publish_odom_tf>true</publish_odom_tf>
       <publish_wheel_tf>false</publish_wheel_tf>
-      <odometry_source>1</odometry_source>
+      <odometry_source>0</odometry_source>
       <!--
         오도메트리 계산 소스:
@@ -47,10 +42,10 @@
           Sim-to-Real 단계에서는 0 (현실적 odom으로 테스트)
       -->
-      <update_rate>50.0</update_rate>
+      <update_rate>${odom_update_rate}</update_rate>
     </plugin>
   </gazebo>
    <gazebo>
     <plugin name="joint_state_publisher" filename="libgazebo_ros_joint_state_publisher.so">
-      <update_rate>50</update_rate>
+      <update_rate>${odom_update_rate}</update_rate>
       <joint_name>left_wheel_joint</joint_name>
       <joint_name>right_wheel_joint</joint_name>
@@ -62,9 +57,9 @@
       <always_on>true</always_on>
       <visualize>false</visualize>
-      <update_rate>5.5</update_rate>
+      <update_rate>${lidar_update_rate}</update_rate>
       <ray>
         <scan>
           <horizontal>
-            <samples>360</samples>
+            <samples>${lidar_samples}</samples>
             <resolution>1.0</resolution>
             <min_angle>-3.14159</min_angle>
@@ -73,6 +68,6 @@
         </scan>
         <range>
-          <min>0.15</min>
-          <max>12.0</max>
+          <min>${lidar_range_min}</min>
+          <max>${lidar_range_max}</max>
           <resolution>0.01</resolution>
         </range>
@@ -80,5 +75,14 @@
           <type>gaussian</type>
           <mean>0.0</mean>
-          <stddev>0.005</stddev>
+          <stddev>${lidar_noise}</stddev>
+          <!--
+            σ = 5mm
+            실제 RPLiDAR A1 노이즈 특성:
+              근거리(1m): σ ≈ 3~5mm
+              중거리(5m): σ ≈ 10~15mm
+              원거리(10m): σ ≈ 30~50mm
+            Gazebo는 거리에 따른 가변 노이즈를 지원하지 않으므로
+            평균적인 값을 사용: 5mm
+          -->
         </noise>
       </ray>
@@ -104,10 +108,10 @@
       <always_on>true</always_on>
       <visualize>false</visualize>
-      <update_rate>30.0</update_rate>
+      <update_rate>${camera_update_rate}</update_rate>
       <camera>
         <horizontal_fov>1.20428</horizontal_fov>
         <image>
-          <width>640</width>
-          <height>480</height>
+          <width>${camera_width}</width>
+          <height>${camera_height}</height>
           <format>B8G8R8</format>
         </image>
@@ -119,5 +123,5 @@
           <type>gaussian</type>
           <mean>0.0</mean>
-          <stddev>0.007</stddev>
+          <stddev>${camera_noise}</stddev>
           <!--
             RGB 이미지 노이즈: σ = 0.007
@@ -142,10 +146,10 @@
       <always_on>true</always_on>
       <visualize>false</visualize>
-      <update_rate>30.0</update_rate>
+      <update_rate>${camera_update_rate}</update_rate>
       <camera>
         <horizontal_fov>1.5184</horizontal_fov>
         <image>
-          <width>640</width>
-          <height>480</height>
+          <width>${camera_width}</width>
+          <height>${camera_height}</height>
           <format>B8G8R8</format>
           <!-- depth 센서도 내부적으로는 이미지 생성 -->
@@ -158,5 +162,5 @@
           <type>gaussian</type>
           <mean>0.0</mean>
-          <stddev>0.005</stddev>
+          <stddev>${depth_noise}</stddev>
         </noise>
       </camera>
@@ -189,11 +193,12 @@
 -->
   <gazebo reference="imu_link">
-    <sensor name="imu" type="imu">
-      <always_on>true</always_on>
-      <update_rate>100.0</update_rate>
+    <gravity>true</gravity>
+    <sensor name="bno055_imu" type="imu">
+      <always_on>true</always_on>
+      <update_rate>${imu_update_rate}</update_rate>
+      <visualize>false</visualize>
       <imu>
         <!-- 각속도 (Gyroscope) 노이즈 -->
         <angular_velocity>
-          <x><noise type="gaussian"><mean>0.0</mean><stddev>0.0002</stddev><bias_mean>0.0000075</bias_mean><bias_stddev>0.0000008</bias_stddev></noise></x>
           <!--
             Bias Random Walk: 느리게 변하는 체계적 편향
@@ -204,10 +209,19 @@
             bias_stddev: 편향이 변하는 속도
           -->
-          <y><noise type="gaussian"><mean>0.0</mean><stddev>0.0002</stddev><bias_mean>0.0000075</bias_mean><bias_stddev>0.0000008</bias_stddev></noise></y>
-          <z><noise type="gaussian"><mean>0.0</mean><stddev>0.0002</stddev><bias_mean>0.0000075</bias_mean><bias_stddev>0.0000008</bias_stddev></noise></z>
+          <x>
+            <noise type="gaussian">
+              <mean>0.0</mean>
+              <stddev>${imu_gyro_noise}</stddev>
+              <bias_mean>0.0</bias_mean>
+              <bias_stddev>4.32e-06</bias_stddev>
+              <dynamic_bias_stddev>4.32e-06</dynamic_bias_stddev>
+              <dynamic_bias_correlation_time>300</dynamic_bias_correlation_time>
+            </noise>
+          </x>
+          <y><noise type="gaussian"><mean>0.0</mean><stddev>${imu_gyro_noise}</stddev><bias_mean>0.0</bias_mean><bias_stddev>4.32e-06</bias_stddev><dynamic_bias_stddev>4.32e-06</dynamic_bias_stddev><dynamic_bias_correlation_time>300</dynamic_bias_correlation_time></noise></y>
+          <z><noise type="gaussian"><mean>0.0</mean><stddev>${imu_gyro_noise}</stddev><bias_mean>0.0</bias_mean><bias_stddev>4.32e-06</bias_stddev><dynamic_bias_stddev>4.32e-06</dynamic_bias_stddev><dynamic_bias_correlation_time>300</dynamic_bias_correlation_time></noise></z>
         </angular_velocity>
         <!-- 선가속도 (Accelerometer) 노이즈 -->
         <linear_acceleration>
-          <x><noise type="gaussian"><mean>0.0</mean><stddev>0.017</stddev><bias_mean>0.1</bias_mean><bias_stddev>0.001</bias_stddev></noise></x>
           <!--
             가속도계 바이어스:
@@ -217,11 +231,19 @@
               → 이것이 EKF에서 가속도계를 "장기 기준"으로만 사용하는 이유!
           -->
-          <y><noise type="gaussian"><mean>0.0</mean><stddev>0.017</stddev><bias_mean>0.1</bias_mean><bias_stddev>0.001</bias_stddev></noise></y>
-          <z><noise type="gaussian"><mean>0.0</mean><stddev>0.017</stddev><bias_mean>0.1</bias_mean><bias_stddev>0.001</bias_stddev></noise></z>
+          <x>
+            <noise type="gaussian">
+              <mean>0.0</mean>
+              <stddev>${imu_accel_noise}</stddev>
+              <bias_mean>0.0</bias_mean>
+              <bias_stddev>3.85e-05</bias_stddev>
+            </noise>
+          </x>
+          <y><noise type="gaussian"><mean>0.0</mean><stddev>${imu_accel_noise}</stddev><bias_mean>0.0</bias_mean><bias_stddev>3.85e-05</bias_stddev></noise></y>
+          <z><noise type="gaussian"><mean>0.0</mean><stddev>${imu_accel_noise}</stddev><bias_mean>0.0</bias_mean><bias_stddev>3.85e-05</bias_stddev></noise></z>
         </linear_acceleration>
       </imu>
-      <plugin name="imu_controller" filename="libgazebo_ros_imu_sensor.so">
-        <ros>
-          <remapping>~/out:=imu/data</remapping>
+      <plugin name="imu_plugin" filename="libgazebo_ros_imu_sensor.so">
+        <ros>
+          <remapping>~/out:=imu/data_raw</remapping>
         </ros>
         <frame_name>imu_link</frame_name>
@@ -239,3 +261,16 @@
   </gazebo>
 -->
+  <gazebo>
+    <plugin name="ground_truth" filename="libgazebo_ros_p3d.so">
+      <ros>
+        <remapping>odom:=/ground_truth/odom</remapping>
+      </ros>
+      <frame_name>odom</frame_name>
+      <body_name>base_footprint</body_name>
+      <update_rate>50</update_rate>
+      <xyz_offset>0 0 0</xyz_offset>
+      <rpy_offset>0 0 0</rpy_offset>
+      <gaussian_noise>0</gaussian_noise>
+    </plugin>
+  </gazebo>
 </robot>

File: src/my_robot_description/urdf/robot_properties.xacro (robot description, xacro)
@@ -11,25 +11,25 @@
   <!-- 프레임 치수 (m 단위!) -->
   <!-- X방향 350mm = 0.350m (전후 길이) -->
-  <xacro:property name="frame_length" value="0.350"/>
+  <xacro:property name="frame_length"     value="0.350"/>
   <!-- Y방향 300mm = 0.300m (좌우 폭) -->
-  <xacro:property name="frame_width" value="0.300"/>
+  <xacro:property name="frame_width"      value="0.300"/>
   <!-- Z방향 240mm = 0.240m (높이) -->
-  <xacro:property name="frame_height" value="0.243"/>
+  <xacro:property name="frame_height"     value="0.243"/>
   <!-- 지상고 57.5mm = 0.0575m -->
   <xacro:property name="ground_clearance" value="0.0575"/>
   <!-- 바퀴 치수 -->
   <!-- 바퀴 반지름 32.5mm -->
-  <xacro:property name="wheel_radius" value="0.0325"/>
+  <xacro:property name="wheel_radius"     value="0.0325"/>
   <!-- 바퀴 폭 20mm -->
-  <xacro:property name="wheel_width" value="0.020"/>
+  <xacro:property name="wheel_width"      value="0.020"/>
   <!-- 좌우 바퀴 사이 거리 345mm -->
   <xacro:property name="wheel_separation" value="0.345"/>
   <!-- 바퀴 X 오프셋: 후방 100mm -->
-  <xacro:property name="wheel_x_offset" value="-0.100"/>
+  <xacro:property name="wheel_x_offset"   value="-0.100"/>
   <!-- 바퀴 Z 오프셋: 하판 아래 25mm -->
-  <xacro:property name="wheel_z_offset" value="-0.025"/>
+  <xacro:property name="wheel_z_offset"   value="-0.025"/>
   <!-- 캐스터 치수 -->
   <!--캐스터 볼 반지름: 12.5mm-->
-  <xacro:property name="caster_radius" value="0.0125"/>
+  <xacro:property name="caster_radius"    value="0.0125"/>
   <!--
     계산:
@@ -42,30 +42,30 @@
   -->
   <!-- 전방 100mm (프레임 앞쪽) -->
-  <xacro:property name="caster_x_offset" value="0.100"/>
+  <xacro:property name="caster_x_offset"      value="0.100"/>
   <!-- 좌우 캐스터 사이 거리: 280mm (Y=±140mm) -->
-  <xacro:property name="caster_y_separation" value="0.280"/>
+  <xacro:property name="caster_y_separation"  value="0.280"/>
   <!-- base_link 원점(하판 바닥)에서 캐스터 볼 중심까지: 45mm -->
-  <xacro:property name="caster_z_offset" value="-0.045"/>
+  <xacro:property name="caster_z_offset"      value="-0.045"/>
   <!-- 질량 (kg) -->
-  <xacro:property name="base_mass" value="4.73"/>
-  <xacro:property name="wheel_mass" value="0.080"/>
-  <xacro:property name="caster_mass" value="0.030"/>
-  <xacro:property name="lidar_mass" value="0.170"/>
-  <xacro:property name="camera_mass" value="0.072"/>
-  <xacro:property name="imu_mass" value="0.010"/>
+  <xacro:property name="base_mass"    value="4.73"/>
+  <xacro:property name="wheel_mass"   value="0.080"/>
+  <xacro:property name="caster_mass"  value="0.030"/>
+  <xacro:property name="lidar_mass"   value="0.170"/>
+  <xacro:property name="camera_mass"  value="0.072"/>
+  <xacro:property name="imu_mass"     value="0.010"/>
   <!-- 센서 위치 -->
-  <xacro:property name="lidar_x" value="-0.130"/>
-  <xacro:property name="lidar_y" value="0.0"/>
-  <xacro:property name="lidar_z" value="0.424"/>
-  <xacro:property name="camera_x" value="0.1875"/>
-  <xacro:property name="camera_y" value="0.0"/>
-  <xacro:property name="camera_z" value="0.2605"/>
-  <xacro:property name="imu_x" value="0.100"/>
-  <xacro:property name="imu_y" value="0.0"/>
-  <xacro:property name="imu_z" value="0.085"/>
+  <xacro:property name="lidar_x"      value="-0.130"/>
+  <xacro:property name="lidar_y"      value="0.0"/>
+  <xacro:property name="lidar_z"      value="0.424"/>
+  <xacro:property name="camera_x"     value="0.1875"/>
+  <xacro:property name="camera_y"     value="0.0"/>
+  <xacro:property name="camera_z"     value="0.2605"/>
+  <xacro:property name="imu_x"        value="0.100"/>
+  <xacro:property name="imu_y"        value="0.0"/>
+  <xacro:property name="imu_z"        value="0.085"/>
   <!-- CoM (무게중심) -->
-  <xacro:property name="base_com_x" value="-0.017"/>
-  <xacro:property name="base_com_y" value="0.0"/>
-  <xacro:property name="base_com_z" value="0.106"/>
+  <xacro:property name="base_com_x"   value="-0.017"/>
+  <xacro:property name="base_com_y"   value="0.0"/>
+  <xacro:property name="base_com_z"   value="0.106"/>
   <!-- 관성 모멘트 매크로 -->
   <!--
@@ -104,3 +104,22 @@
     </inertial>
   </xacro:macro>
+  <!-- 노이즈 파라미터 (Day 53 Allan Variance 결과) -->
+    <!-- Diff Drive 파라미터 -->
+    <xacro:property name="odom_update_rate"     value="50"/>
+    <!-- LiDAR 노이즈 -->
+    <xacro:property name="lidar_noise"          value="0.005"/>
+    <xacro:property name="lidar_samples"        value="360"/>
+    <xacro:property name="lidar_update_rate"    value="5.5"/>
+    <xacro:property name="lidar_range_min"      value="0.15"/>
+    <xacro:property name="lidar_range_max"      value="12.0"/>
+    <!-- Camera 노이즈 -->
+    <xacro:property name="camera_noise"         value="0.007"/>
+    <xacro:property name="depth_noise"          value="0.005"/>
+    <xacro:property name="camera_update_rate"   value="30"/>
+    <xacro:property name="camera_width"         value="640"/>
+    <xacro:property name="camera_height"        value="480"/>
+    <!-- IMU 노이즈 -->
+    <xacro:property name="imu_gyro_noise"       value="0.000193"/>
+    <xacro:property name="imu_accel_noise"      value="0.0168"/>
+    <xacro:property name="imu_update_rate"      value="100"/>
 </robot>

File: src/my_robot_description/urdf/robot_wheels.xacro (robot description, xacro)
@@ -12,9 +12,4 @@
     -->
     <joint name="${prefix}_wheel_joint" type="continuous">
-      <!--
-        ${prefix}_wheel_joint
-          → "left_wheel_joint" 또는 "right_wheel_joint"
-          → 문자열 조합이 가능
-      -->
       <parent link="base_link"/>
       <child link="${prefix}_wheel"/>
@@ -65,5 +60,4 @@
       </collision>
       <xacro:cylinder_inertia m="${wheel_mass}" r="${wheel_radius}" h="${wheel_width}"/>
-      <!-- ⭐ 관성 모멘트 매크로 호출 → robot_properties.xacro에서 정의한 매크로 -->
     </link>
     <!-- Gazebo 마찰 설정 -->
@@ -72,23 +66,24 @@
       <mu1>1.0</mu1>
       <mu2>1.0</mu2>
-      <kp>1000000.0</kp>
-      <kd>10.0</kd>
+      <!--
+        바퀴 마찰 계수
+          μ=1.0: 고무 바퀴 (높은 마찰!)
+        이 값이 너무 작으면:
+          → 바퀴 공회전! → 오도메트리가 실제보다 앞서감!
+          → Sim-to-Real Gap 원인!
+      -->
+      <kp>1e6</kp>
+      <kd>100</kd>
+      <!--
+        접촉 강성 (kp)과 감쇠 (kd)
+          → 바퀴-바닥 접촉의 "딱딱함"
+          → kp 너무 크면: 진동
+          → kp 너무 작면: 바퀴가 바닥에 파묻힘
+      -->
     </gazebo>
   </xacro:macro>
   <!-- 매크로 호출 — 바퀴 2개 생성! -->
   <xacro:wheel prefix="left" y_reflect="1"/>
-  <!--
-    이 한 줄로 생성되는 것:
-      ✅ left_wheel_joint (continuous, Y=+0.172.5)
-      ✅ left_wheel (link with visual/collision/inertial)
-      ✅ Gazebo 마찰 설정
-  -->
   <xacro:wheel prefix="right" y_reflect="-1"/>
-  <!--
-    이 한 줄로 생성되는 것:
-      ✅ right_wheel_joint (continuous, Y=-0.172.5)
-      ✅ right_wheel (link with visual/collision/inertial)
-      ✅ Gazebo 마찰 설정
-  -->
   <!-- ============================================ -->
   <!-- 캐스터 매크로 정의 -->
@@ -141,11 +136,11 @@
     <gazebo reference="${prefix}_caster_link">
       <material>Gazebo/DarkGrey</material>
-      <mu1>0.001</mu1>
-      <mu2>0.001</mu2>
+      <mu1>0.01</mu1>
+      <mu2>0.01</mu2>
       <!--
         ⭐ 핵심: 마찰이 거의 0!
         mu = 0.001:
           구동 바퀴: mu = 1.0 (높은 마찰 = 접지력)
-          캐스터: mu = 0.001 (거의 무마찰 = 자유 미끄러짐)
+          캐스터: mu = 0.01 (거의 무마찰 = 자유 미끄러짐)
         왜?
           차동 구동의 회전 원리:
@@ -154,14 +149,7 @@
               캐스터 마찰이 높으면 → 회전 못 함!
       -->
-      <kp>1000000.0</kp>
-      <kd>100.0</kd>
-      <!--
-        kp: 접촉 강성 (높아야 바닥을 안 뚫음)
-        kd: 접촉 감쇠 (바운스 방지)
-        kd를 10→100으로 올림:
-          캐스터가 작고 가벼워서 진동이 생기기 쉬움
-          감쇠를 높여서 안정화!
-      -->
-    </gazebo>    \
+      <kp>1e6</kp>
+      <kd>100</kd>
+    </gazebo>
   </xacro:macro>
   <!-- 캐스터 매크로 호출 — 2개 생성! -->
