Commit message: Day 59

File: src/my_robot_description/urdf/robot_gazebo.xacro (robot description, xacro)
@@ -212,13 +212,30 @@
             <noise type="gaussian">
               <mean>0.0</mean>
-              <stddev>${imu_gyro_noise}</stddev>
-              <bias_mean>0.0</bias_mean>
-              <bias_stddev>4.32e-06</bias_stddev>
-              <dynamic_bias_stddev>4.32e-06</dynamic_bias_stddev>
+              <stddev>${imu_gyro_noise_stddev}</stddev>
+              <bias_mean>${imu_gyro_noise_bias_mean}</bias_mean>
+              <bias_stddev>${imu_gyro_noise_bias_stddev}</bias_stddev>
+              <dynamic_bias_stddev>${imu_gyro_noise_dynamic_bias_stddev}</dynamic_bias_stddev>
               <dynamic_bias_correlation_time>300</dynamic_bias_correlation_time>
             </noise>
           </x>
-          <y><noise type="gaussian"><mean>0.0</mean><stddev>${imu_gyro_noise}</stddev><bias_mean>0.0</bias_mean><bias_stddev>4.32e-06</bias_stddev><dynamic_bias_stddev>4.32e-06</dynamic_bias_stddev><dynamic_bias_correlation_time>300</dynamic_bias_correlation_time></noise></y>
-          <z><noise type="gaussian"><mean>0.0</mean><stddev>${imu_gyro_noise}</stddev><bias_mean>0.0</bias_mean><bias_stddev>4.32e-06</bias_stddev><dynamic_bias_stddev>4.32e-06</dynamic_bias_stddev><dynamic_bias_correlation_time>300</dynamic_bias_correlation_time></noise></z>
+          <y>
+            <noise type="gaussian">
+              <mean>0.0</mean>
+              <stddev>${imu_gyro_noise_stddev}</stddev>
+              <bias_mean>${imu_gyro_noise_bias_mean}</bias_mean>
+              <bias_stddev>${imu_gyro_noise_bias_stddev}</bias_stddev>
+              <dynamic_bias_stddev>${imu_gyro_noise_dynamic_bias_stddev}</dynamic_bias_stddev>
+              <dynamic_bias_correlation_time>300</dynamic_bias_correlation_time>
+            </noise>
+          </y>
+          <z><noise type="gaussian">
+            <mean>0.0</mean>
+            <stddev>${imu_gyro_noise_stddev}</stddev>
+            <bias_mean>${imu_gyro_noise_bias_mean}</bias_mean>
+            <bias_stddev>${imu_gyro_noise_bias_stddev}</bias_stddev>
+            <dynamic_bias_stddev>${imu_gyro_noise_dynamic_bias_stddev}</dynamic_bias_stddev>
+            <dynamic_bias_correlation_time>300</dynamic_bias_correlation_time>
+          </noise>
+        </z>
         </angular_velocity>
         <!-- 선가속도 (Accelerometer) 노이즈 -->
@@ -234,11 +251,25 @@
             <noise type="gaussian">
               <mean>0.0</mean>
-              <stddev>${imu_accel_noise}</stddev>
-              <bias_mean>0.0</bias_mean>
-              <bias_stddev>3.85e-05</bias_stddev>
+              <stddev>${imu_accel_noise_stddev}</stddev>
+              <bias_mean>${imu_accel_noise_bias_mean}</bias_mean>
+              <bias_stddev>${imu_accel_noise_bias_stddev}</bias_stddev>
             </noise>
           </x>
-          <y><noise type="gaussian"><mean>0.0</mean><stddev>${imu_accel_noise}</stddev><bias_mean>0.0</bias_mean><bias_stddev>3.85e-05</bias_stddev></noise></y>
-          <z><noise type="gaussian"><mean>0.0</mean><stddev>${imu_accel_noise}</stddev><bias_mean>0.0</bias_mean><bias_stddev>3.85e-05</bias_stddev></noise></z>
+          <y>
+            <noise type="gaussian">
+              <mean>0.0</mean>
+              <stddev>${imu_accel_noise_stddev}</stddev>
+              <bias_mean>${imu_accel_noise_bias_mean}</bias_mean>
+              <bias_stddev>${imu_accel_noise_bias_stddev}</bias_stddev>
+            </noise>
+          </y>
+          <z>
+            <noise type="gaussian">
+              <mean>0.0</mean>
+              <stddev>${imu_accel_noise_stddev}</stddev>
+              <bias_mean>${imu_accel_noise_bias_mean}</bias_mean>
+              <bias_stddev>${imu_accel_noise_bias_stddev}</bias_stddev>
+              </noise>
+            </z>
         </linear_acceleration>
       </imu>

File: src/my_robot_description/urdf/robot_properties.xacro (robot description, xacro)
@@ -120,6 +120,11 @@
     <xacro:property name="camera_height"        value="480"/>
     <!-- IMU 노이즈 -->
-    <xacro:property name="imu_gyro_noise"       value="0.000193"/>
-    <xacro:property name="imu_accel_noise"      value="0.0168"/>
+    <xacro:property name="imu_gyro_noise_stddev"                value="0.000199"/>
+    <xacro:property name="imu_gyro_noise_bias_mean"             value="0.0"/>
+    <xacro:property name="imu_gyro_noise_bias_stddev"           value="9.95e-07"/>
+    <xacro:property name="imu_gyro_noise_dynamic_bias_stddev"   value="9.95e-07"/>
+    <xacro:property name="imu_accel_noise_stddev"               value="0.0171"/>
+    <xacro:property name="imu_accel_noise_bias_mean"            value="0.0"/>
+    <xacro:property name="imu_accel_noise_bias_stddev"          value="2.28e-04"/>
     <xacro:property name="imu_update_rate"      value="100"/>
 </robot>
